File: Pcb/Kicad/PCB_Designs-master/Kidcad_basic/beginer/beginer.kicad_pcb (KiCad board)
At the start: 2 copper layers, 88 x 41.9 mm, 16 parts, among them J1 PINHD_1x1_Female, J10 PINHD_1x1_Female, J11 PINHD_1x1_Female, J12 PINHD_1x1_Female, J2 PINHD_1x1_Female, J3 PINHD_1x1_Female, J4 PINHD_1x1_Female, J5 PINHD_1x1_Female, J6 PINHD_1x1_Female, J7 PINHD_1x1_Female, J8 PINHD_1x1_Female, J9 PINHD_1x1_Female, SW1 SW_DPDT_x2

Commit message: update file kicad
Parts:
- removed BT1: Battery_Cell, Battery:BatteryHolder_Keystone_1058_1x2032
- removed J10, J11, J12, J8, J9: PINHD_1x1_Female, Connector_PinSocket_2.54mm:PinSocket_1x01_P2.54mm_Vertical
- removed SW1: SW_DPDT_x2, Button_Switch_THT:SW_TH_Tactile_Omron_B3F-10xx
- added C1: 10U, Capacitor_THT:C_Disc_D3.0mm_W1.6mm_P2.50mm, F.Cu at (110.0, 87.8)
- added C2: 0.1U, Capacitor_THT:C_Disc_D3.0mm_W1.6mm_P2.50mm, F.Cu at (110.0, 110.3)
- added C3: 1U, Capacitor_THT:C_Disc_D3.0mm_W1.6mm_P2.50mm, F.Cu at (135.0, 77.5)
- added G***: LOGO, EG1218:LUFFY, B.Cu at (131.0, 90.0)
- added R2: 330, Resistor_THT:R_Axial_DIN0204_L3.6mm_D1.6mm_P7.62mm_Horizontal, F.Cu at (100.0, 105.3)
- added R3: 560, Resistor_THT:R_Axial_DIN0204_L3.6mm_D1.6mm_P7.62mm_Horizontal, F.Cu at (105.0, 97.7)
- added S1: EG1218, EG1218:SW_EG1218, F.Cu at (100.0, 82.8)
- added U1: LM317_TO-220, Package_TO_SOT_THT:TO-220-3_Vertical, F.Cu at (120.0, 100.3)
- added U2: LM7805_TO220, Package_TO_SOT_THT:TO-220-3_Vertical, F.Cu at (120.0, 75.3)
- J1: value PINHD_1x1_Female -> Barrel_Jack_Switch; footprint Connector_PinSocket_2.54mm:PinSocket_1x01_P2.54mm_Vertical -> Connector_BarrelJack:BarrelJack_Horizontal
- J2, J7: value PINHD_1x1_Female -> Screw_Terminal_2_P3.50mm; footprint Connector_PinSocket_2.54mm:PinSocket_1x01_P2.54mm_Vertical -> TerminalBlock_Phoenix:TerminalBlock_Phoenix_PT-1,5-2-3.5-H_1x02_P3.50mm_Horizontal
- J3, J5: value PINHD_1x1_Female -> PINHD_1x2_Male; footprint Connector_PinSocket_2.54mm:PinSocket_1x01_P2.54mm_Vertical -> Connector_PinHeader_2.54mm:PinHeader_1x02_P2.54mm_Vertical
- J4, J6: value PINHD_1x1_Female -> PINHD_1x3_Male; footprint Connector_PinSocket_2.54mm:PinSocket_1x01_P2.54mm_Vertical -> Connector_PinHeader_2.54mm:PinHeader_1x03_P2.54mm_Vertical
- R1: value R -> 330
- moved J2 73.8 mm to (155.0, 103.8), turned to 90 degrees
- moved J4 65.3 mm to (145.0, 105.3), turned to 180 degrees
- moved J7 50.0 mm to (155.0, 78.8), turned to 90 degrees
- moved J1 46.2 mm to (111.0, 70.3)
- moved J6 37.6 mm to (148.0, 88.5), turned to 180 degrees
- moved J5 36.7 mm to (140.0, 100.3)
- moved J3 33.2 mm to (142.0, 77.5), turned to 180 degrees
- moved D1 23.7 mm to (125.0, 87.5)
- moved R1 10.7 mm to (130.0, 107.6)
Connections:
- D1 pad 1: Net-(BT1--) -> GND
- D1 pad 2: Net-(D1-A) -> Net-(R2-+)
- J1 pad 1: /net1 -> /PWR_input
- J2 pad 1: /net1 -> GND
- J3 pad 1: /net1 -> GND
- J4 pad 1: /net1 -> /5V
- J5 pad 1: /net3 -> GND
- J6 pad 1: /net3 -> /5V
- J7 pad 1: /net1 -> GND
- R1 pad 1: Net-(D1-A) -> Net-(R1-+)
- R1 pad 2: Net-(SW1A-A) -> /3.3V
Routing:
- net /PWR_output: track 0.00 -> 80.4 mm
- net /net1: track 75.9 -> 0.00 mm
- net /3.3V: track 0.00 -> 71.9 mm
- net Net-(R2-+): track 0.00 -> 70.2 mm
- net /12V: track 0.00 -> 64.5 mm
- net /5V: track 0.00 -> 54.4 mm
- net Net-(BT1-+): track 51.9 -> 0.00 mm
- net Net-(BT1--): track 47.6 -> 0.00 mm
- net /net3: track 40.0 -> 0.00 mm
- net Net-(R1-+): track 0.00 -> 33.1 mm
- net /PWR_input: track 0.00 -> 26.5 mm
- net Net-(SW1A-A): track 22.3 -> 0.00 mm
- net /net2: track 15.0 -> 0.00 mm
- net Net-(D1-A): track 14.5 -> 0.00 mm
- added copper zone on B.Cu, net GND
Other:
- board size 88 x 41.9 mm -> 70 x 50 mm
- board text added: "OFF"
- board text added: "ON"
