File: Pcb/Kicad/PCB_Designs-master/Kidcad_basic/beginer/sheet3.kicad_sch (KiCad schematic)
At the start: 2 parts, among them J13 PINHD_1x1_Female, J14 PINHD_1x1_Female

Commit message: update file kicad
Parts:
- removed J13, J14: PINHD_1x1_Female, Connector_PinSocket_2.54mm:PinSocket_1x01_P2.54mm_Vertical, symbol PCM_SL_Pin_Headers:PINHD_1x1_Female
- added C1, C2, C3: C, symbol PCM_Elektuur:C
- added D1: LED, LED_THT:LED_D5.0mm, symbol PCM_SL_Devices:LED
- added J1, J2: PINHD_1x2_Male, Connector_PinHeader_2.54mm:PinHeader_1x02_P2.54mm_Vertical, symbol PCM_SL_Pin_Headers:PINHD_1x2_Male
- added J3, J4: PINHD_1x3_Male, Connector_PinHeader_2.54mm:PinHeader_1x03_P2.54mm_Vertical, symbol PCM_SL_Pin_Headers:PINHD_1x3_Male
- added J5: Screw_Terminal_2_P3.50mm, TerminalBlock_Phoenix:TerminalBlock_Phoenix_PT-1,5-2-3.5-H_1x02_P3.50mm_Horizontal, symbol PCM_SL_Screw_Terminal:Screw_Terminal_2_P3.50mm
- added J7: Barrel_Jack_Switch, symbol Connector:Barrel_Jack_Switch
- added R1, R2, R3: R, symbol PCM_Elektuur:R
- added S1: EG1218, EG1218:SW_EG1218, symbol EG1218:EG1218
- added U1, U2: LM7805_TO220, Package_TO_SOT_THT:TO-220-3_Vertical, symbol Regulator_Linear:LM7805_TO220
