File: Pcb/Kicad/PCB_Designs-master/Kidcad_basic/beginer/sheetnew.kicad_sch (KiCad schematic)
At the start: 2 parts, among them J15 PINHD_1x1_Female, J16 PINHD_1x1_Female

Commit message: update file kicad
Parts:
- removed J15, J16: PINHD_1x1_Female, Connector_PinSocket_2.54mm:PinSocket_1x01_P2.54mm_Vertical, symbol PCM_SL_Pin_Headers:PINHD_1x1_Female
Changed lines of the file:
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@@
 	(generator_version "8.0")
 	(paper "A4")
-	(wire
-		(pts
-			(xy 112.522 102.87) (xy 151.892 102.87)
-		)
-		(stroke
-			(width 0)
-			(type default)
-		)
-	)
-	(label "net3"
-		(at 132.334 102.87 0)
-		(fields_autoplaced yes)
-		(effects
-			(font
-				(size 1.27 1.27)
-			)
-			(justify left bottom)
-		)
-	)
-	(symbol
-		(lib_id "PCM_SL_Pin_Headers:PINHD_1x1_Female")
-		(at 155.702 102.87 0)
-		(unit 1)
-		(exclude_from_sim no)
-		(in_bom yes)
-		(on_board yes)
-		(dnp no)
-		(fields_autoplaced yes)
-		(property "Reference" "J16"
-			(at 159.004 101.5999 0)
-			(effects
-				(font
-					(size 1.27 1.27)
-				)
-				(justify left)
-			)
-		)
-		(property "Value" "PINHD_1x1_Female"
-			(at 159.004 104.1399 0)
-			(effects
-				(font
-					(size 1.27 1.27)
-				)
-				(justify left)
-			)
-		)
-		(property "Footprint" "Connector_PinSocket_2.54mm:PinSocket_1x01_P2.54mm_Vertical"
-			(at 158.242 93.98 0)
-			(effects
-				(font
-					(size 1.27 1.27)
-				)
-				(hide yes)
-			)
-		)
-		(property "Datasheet" ""
-			(at 155.702 96.52 0)
-			(effects
-				(font
-					(size 1.27 1.27)
-				)
-				(hide yes)
-			)
-		)
-		(property "Description" "Pin Header female with pin space 2.54mm. Pin Count -1"
-			(at 155.702 102.87 0)
-			(effects
-				(font
-					(size 1.27 1.27)
-				)
-				(hide yes)
-			)
-		)
-		(pin "1"
-		)
-		(instances
-			(project "beginer"
-				(path "/1c1ee748-2851-4e44-9ba4-33b83351618f/0e2d05fb-be23-4f46-b309-550af2bbc1e9"
-					(reference "J16")
-					(unit 1)
-				)
-			)
-		)
-	)
-	(symbol
-		(lib_id "PCM_SL_Pin_Headers:PINHD_1x1_Female")
-		(at 108.712 102.87 180)
-		(unit 1)
-		(exclude_from_sim no)
-		(in_bom yes)
-		(on_board yes)
-		(dnp no)
-		(fields_autoplaced yes)
-		(property "Reference" "J15"
-			(at 108.457 96.52 0)
-			(effects
-				(font
-					(size 1.27 1.27)
-				)
-			)
-		)
-		(property "Value" "PINHD_1x1_Female"
-			(at 108.457 99.06 0)
-			(effects
-				(font
-					(size 1.27 1.27)
-				)
-			)
-		)
-		(property "Footprint" "Connector_PinSocket_2.54mm:PinSocket_1x01_P2.54mm_Vertical"
-			(at 106.172 111.76 0)
-			(effects
-				(font
-					(size 1.27 1.27)
-				)
-				(hide yes)
-			)
-		)
-		(property "Datasheet" ""
-			(at 108.712 109.22 0)
-			(effects
-				(font
-					(size 1.27 1.27)
-				)
-				(hide yes)
-			)
-		)
-		(property "Description" "Pin Header female with pin space 2.54mm. Pin Count -1"
-			(at 108.712 102.87 0)
-			(effects
-				(font
-					(size 1.27 1.27)
-				)
-				(hide yes)
-			)
-		)
-		(pin "1"
-		)
-		(instances
-			(project "beginer"
-				(path "/1c1ee748-2851-4e44-9ba4-33b83351618f/0e2d05fb-be23-4f46-b309-550af2bbc1e9"
-					(reference "J15")
-					(unit 1)
-				)
-			)
-		)
-	)
 	(sheet
 		(at 231.648 110.744)
