File: Pcb/Kicad/PCB_Designs-master/STM32F103_InverterVCU/inverter_vcu.kicad_pcb (KiCad board)
At the start: 2 copper layers, 69.9 x 65.4 mm, 53 parts, among them J1 Conn_01x03_Male, J10 Conn_01x02_Male, J11 Conn_01x04_Male, J12 DB9_Male_MountingHoles, J13 Conn_01x02_Male, J14 Conn_01x03_Male, J15 Conn_01x07_Male, J16 Conn_01x07_Male, J17 Conn_01x03_Male, J2 Conn_01x07_Male, J3 Conn_01x02_Male, J4 Conn_01x02_Male, J5 Conn_01x02_Male, J6 Conn_01x01_Male, J7 Conn_01x01_Male, J8 Conn_01x04_Male, J9 Conn_01x03_Male, SW1 SW_Push, U1 STM32F103C8Tx, U2 MCP2551-I-SN, U3 LM7805_TO220, U4 AMS1117-3.3, Y1 Crystal

Commit message: update code
Parts:
- removed the G*** at (162.9, 108.0)
- added G***: LOGO, EG1218:LUFFY, F.Cu at (166.0, 111.0)
Other:
- board text added: "3.3V"
- board text added: "MISO"
- board text added: "MOSI"
- board text added: "SCK"
- board text added: "SWCLK"
- board text removed: "Vegapod Hyperloop"
