File: Pcb/Kicad/PCB_Designs-master/STM32F103_board/f103_V2.kicad_pcb (KiCad board)
At the start: 2 copper layers, 84.4 x 79.2 mm, 60 parts, among them J1 Conn_01x04_Male, J10 DB9_Male_MountingHoles, J11 Conn_01x03_Male, J12 Conn_01x02_Male, J2 Conn_01x03_Male, J3 Conn_01x06_Male, J4 Conn_02x02_Odd_Even, J5 Conn_01x03_Male, J6 Conn_01x02_Male, J7 Conn_02x05_Top_Bottom, J8 Conn_01x04_Male, J9 USB_B_Micro, SW1 SW_Push, SW2 SW_SPDT, SW3 SW_Push, U1 AMS1117-3.3, U2 74LS47, U3 SA39-12EWA, U4 STM32F103C8Tx, U5 MCP2551-I-SN, Y1 Crystal

Commit message: update code
Parts:
- removed G***: LOGO, BluePill_slave:logo6
- removed REF** (x3): MountingHole_3.2mm_M3, MountingHole:MountingHole_3.2mm_M3
- C6: value 100nF -> 10uF
- J11: footprint Connector_Phoenix_GMSTB:PhoenixContact_GMSTBVA_2,5_3-G-7,62_1x03_P7.62mm_Vertical -> Connector_Phoenix_MC:PhoenixContact_MCV_1,5_3-G-3.81_1x03_P3.81mm_Vertical
Routing:
- net (no net): track 0.00 -> 49.5 mm
- net unconnected-(J10-PAD-Pad0)_1: track 34.2 -> 0.00 mm
- net unconnected-(J9-Shield-Pad6): track 15.3 -> 0.00 mm
- net VBUS: track 219.3 -> 219.9 mm
Other:
- board text removed: "Designed by Varad V1.2"
- board text removed: "Powering the board -Power Port -DB9 conn -USB Do not power the board with two ports at same time Use only one power source"
- board text removed: "Vegapod Hyperloop"
