File: Pcb/Kicad/PCB_Designs-master/STM32F103_board/f103_V2.kicad_sch (KiCad schematic)
At the start: 56 parts, among them J1 Conn_01x04_Male, J10 DB9_Male_MountingHoles, J11 Conn_01x03_Male, J12 Conn_01x02_Male, J2 Conn_01x03_Male, J3 Conn_01x06_Male, J4 Conn_02x02_Odd_Even, J5 Conn_01x03_Male, J6 Conn_01x02_Male, J7 Conn_02x05_Top_Bottom, J8 Conn_01x04_Male, J9 USB_B_Micro, SW1 SW_Push, SW2 SW_SPDT, SW3 SW_Push, U1 AMS1117-3.3, U2 74LS47, U3 SA39-12EWA, U4 STM32F103C8Tx, U5 MCP2551-I-SN, Y1 Crystal

Commit message: update code
Connections:
- no-connect marks 12 -> 14
